Commit message: Error rectified

File: robot_model/mm_400_panda/urdf/xacros/mp_400_body.xacro (robot description, xacro)
@@ -3,15 +3,15 @@
   <xacro:macro name="mp_400_base" params="name">
     <link name="${name}">
-      <inertial>
-        <mass value="250"/>
-        <origin xyz="0 0 0" />
-         <inertia ixx="5.652232699207" ixy="0.009719934438" ixz="1.293988226423"
-                 iyy="5.669473158652" iyz="0.007379583694"
-                 izz="5.683196351726" />
-      </inertial>
+  <inertial>
+        <mass value="125" />
+        <origin xyz="0 0 0" rpy="0 0 0"/>
+        <inertia ixx="1.71402" ixy="0.0" ixz="0.0"
+                 iyy="0.8856" iyz="0.0"
+                 izz="2.5725" />
+</inertial>
       <visual name='body'>
       <origin xyz="0.0 0.0 0." rpy="0 0 1.57" />
         <geometry>
-            <mesh filename="package://neo_mm_400/robot_model/mm_400_panda/meshes/top.dae" scale="0.001 0.001 0.001"/>
+            <mesh filename="package://neo_mm_400/robot_model/mm_400_panda/meshes/MP-400-BODY.dae" scale="0.001 0.001 0.001"/>
         <!--cylinder length="0.381" radius="0.2545"/-->
         <!--box size="0.445 0.277 0.17"/-->
@@ -21,5 +21,5 @@
         <origin xyz="0.0 0.0 0.0" rpy="0 0 1.57" />
         <geometry>
-            <mesh filename="package://neo_mm_400/robot_model/mm_400_panda/meshes/top.dae" scale="0.001 0.001 0.001"/>
+            <mesh filename="package://neo_mm_400/robot_model/mm_400_panda/meshes/MP-400-BODY.dae" scale="0.001 0.001 0.001"/>
           <!--cylinder length="0.381" radius="0.2545"/-->
         </geometry>
