Commit message: Error rectified-1

File: robot_model/mm_400_panda/urdf/xacros/cabinet.xacro (robot description, xacro)
@@ -19,5 +19,5 @@
         <origin xyz="0 0 0" rpy="0 0 -1.5708" />
         <geometry>
-            <mesh filename="package://neo_simulation/robots/mm_400/meshes/top.dae" scale="0.001 0.001 0.001"/>
+            <mesh filename="package://neo_mm_400/robot_model/mm_400_panda/meshes/top.dae" scale="0.001 0.001 0.001"/>
         </geometry>
       </visual>
@@ -25,5 +25,5 @@
         <origin xyz="0. 0. 0" rpy="0 0 0" />
         <geometry>
-            <mesh filename="package://neo_simulation/robots/mm_400/meshes/top.dae" scale="0.001 0.001 0.001"/>
+            <mesh filename="package://neo_mm_400/robot_model/mm_400_panda/meshes/top.dae" scale="0.001 0.001 0.001"/>
         </geometry>
       </collision>

File: robot_model/mm_400_panda/urdf/xacros/sick_laser.xacro (robot description, xacro)
@@ -18,5 +18,5 @@
 <!--       <origin xyz="0 0 -0.11" rpy="-1.57 0 3.14" />
         <geometry>
-        <mesh filename="package://neo_simulation/robots/mp_400/meshes/SICK-S300.dae" scale="0.001 0.001 0.001" />
+        <mesh filename="package://neo_mm_400/robot_model/mm_400_panda/meshes/SICK-S300.dae" scale="0.001 0.001 0.001" />
         </geometry>
       </visual>
@@ -24,5 +24,5 @@
         <origin xyz="0 0 -0.11" rpy="-1.57 0 3.14" />
         <geometry>
-        <mesh filename="package://neo_simulation/robots/mp_400/meshes/SICK-S300.dae" scale="0.001 0.001 0.001" />
+        <mesh filename="package://neo_mm_400/robot_model/mm_400_panda/meshes/meshes/SICK-S300.dae" scale="0.001 0.001 0.001" />
         </geometry>
       </collision> -->
