Commit message: Links to the models have been changed

File: robot_model/mm_400.urdf.xacro (robot description, xacro)
@@ -2,19 +2,19 @@
 <!-- Materials -->
 <robot xmlns:xacro="http://www.ros.org/wiki/xacro" name="mm_400">
-<xacro:include filename="$(find neo_simulation)/robots/mp_400/xacros/mp_400_gazebo.xacro" />
+<xacro:include filename="$(find neo_mm_400)/robot_model/xacros/mp_400_gazebo.xacro" />
 <!--++++++++++++++++++++++++++++++base_link++++++++++++++++++++++++++++++++++++++++++++++++++++-->
 <!--++++++++++++++++++++body++++++++++++++++++++++++++++-->
-<xacro:include filename="$(find neo_simulation)/robots/mm_400/urdf/xacros/mp_400_body.xacro" />
+<xacro:include filename="$(find neo_mm_400)/robot_model/urdf/xacros/mp_400_body.xacro" />
 <!--+++++++++++++++++++castor_wheel_link++++++++++++++++++++++++-->
-<xacro:include filename="$(find neo_simulation)/robots/mm_400/urdf/xacros/mp_400_caster_wheel.xacro" />
+<xacro:include filename="$(find neo_mm_400)/robot_model/urdf/xacros/mp_400_caster_wheel.xacro" />
 <!--+++++++++++++++++++left_wheel_link++++++++++++++++++++++++-->
-<xacro:include filename="$(find neo_simulation)/robots/mm_400/urdf/xacros/mp_400_fixed_wheel_left.xacro" />
+<xacro:include filename="$(find neo_mm_400)/robot_model/urdf/xacros/mp_400_fixed_wheel_left.xacro" />
 <!--+++++++++++++++++++right_wheel_link++++++++++++++++++++++++-->
-<xacro:include filename="$(find neo_simulation)/robots/mm_400/urdf/xacros/mp_400_fixed_wheel_right.xacro" />
+<xacro:include filename="$(find neo_mm_400)/robot_model/urdf/xacros/mp_400_fixed_wheel_right.xacro" />
 <!--+++++++++++++++++++cabinet++++++++++++++++++++++++-->
-<xacro:include filename="$(find neo_simulation)/robots/mm_400/urdf/xacros/cabinet.xacro" />
-<xacro:include filename="$(find neo_simulation)/robots/mm_400/urdf/prbt_macro.xacro" />
+<xacro:include filename="$(find neo_mm_400)/robot_model/urdf/xacros/cabinet.xacro" />
+<xacro:include filename="$(find neo_mm_400)/robot_model/urdf/prbt_macro.xacro" />
  <!-- SENSORS -->
-<xacro:include filename="$(find neo_simulation)/robots/mm_400/urdf/xacros/sick_laser.xacro" />
+<xacro:include filename="$(find neo_mm_400)/robot_model/urdf/xacros/sick_laser.xacro" />
   <xacro:mp_400_base name="base_link">
   </xacro:mp_400_base>

File: robot_model/urdf/prbt_macro.xacro (robot description, xacro)
@@ -36,5 +36,5 @@
         <origin xyz="0 0 0" rpy="0 0 0" />
         <geometry>
-          <mesh filename="package://neo_simulation/robots/mm_400/meshes/foot.dae" />
+          <mesh filename="package://neo_mm_400/robot_model/mm_400/meshes/foot.dae" />
         </geometry>
       </visual>
@@ -65,5 +65,5 @@
         <origin xyz="0 0 0" rpy="0 0 0" />
         <geometry>
-          <mesh filename="package://neo_simulation/robots/mm_400/meshes/link_1.dae" />
+          <mesh filename="package://neo_mm_400/robot_model/mm_400/meshes/link_1.dae" />
         </geometry>
       </visual>
@@ -105,5 +105,5 @@
         <origin xyz="0 0 0" rpy="0 0 -${pi/3}" />
         <geometry>
-          <mesh filename="package://neo_simulation/robots/mm_400/meshes/link_2.dae" />
+          <mesh filename="package://neo_mm_400/robot_model/mm_400/meshes/link_2.dae" />
         </geometry>
       </visual>
@@ -139,5 +139,5 @@
         <origin xyz="0 0 0" rpy="0 0 ${pi}" />
         <geometry>
-          <mesh filename="package://neo_simulation/robots/mm_400/meshes/link_3.dae" />
+          <mesh filename="package://neo_mm_400/robot_model/mm_400/meshes/link_3.dae" />
         </geometry>
       </visual>
@@ -179,5 +179,5 @@
         <origin xyz="0 0 0" rpy="0 0 0" />
         <geometry>
-          <mesh filename="package://neo_simulation/robots/mm_400/meshes/link_4.dae" />
+          <mesh filename="package://neo_mm_400/robot_model/mm_400/meshes/link_4.dae" />
         </geometry>
       </visual>
@@ -213,5 +213,5 @@
         <origin xyz="0 0 0" rpy="0 0 0" />
         <geometry>
-          <mesh filename="package://neo_simulation/robots/mm_400/meshes/link_5.dae"/>
+          <mesh filename="package://neo_mm_400/robot_model/mm_400/meshes/link_5.dae"/>
         </geometry>
       </visual>
@@ -266,5 +266,5 @@
         <origin xyz="0 0 0" rpy="0 0 0" />
         <geometry>
-          <mesh filename="package://neo_simulation/robots/mm_400/meshes/flange.dae"/>
+          <mesh filename="package://neo_mm_400/robot_model/mm_400/meshes/flange.dae"/>
         </geometry>
       </visual>

File: robot_model/urdf/xacros/cabinet.xacro (robot description, xacro)
@@ -19,5 +19,5 @@
         <origin xyz="0 0 0" rpy="0 0 -1.5708" />
         <geometry>
-            <mesh filename="package://neo_simulation/robots/mm_400/meshes/top.dae" scale="0.001 0.001 0.001"/>
+            <mesh filename="package://neo_mm_400/robot_model/mm_400/meshes/top.dae" scale="0.001 0.001 0.001"/>
         </geometry>
       </visual>
@@ -25,5 +25,5 @@
         <origin xyz="0. 0. 0" rpy="0 0 0" />
         <geometry>
-            <mesh filename="package://neo_simulation/robots/mm_400/meshes/top.dae" scale="0.001 0.001 0.001"/>
+            <mesh filename="package://neo_mm_400/robot_model/mm_400/meshes/top.dae" scale="0.001 0.001 0.001"/>
         </geometry>
       </collision>

File: robot_model/urdf/xacros/mp_400_body.xacro (robot description, xacro)
@@ -13,5 +13,5 @@
       <origin xyz="0.0 0.0 0." rpy="0 0 1.57" />
         <geometry>
-            <mesh filename="package://neo_simulation/robots/mm_400/meshes/MP-400-BODY.dae" scale="0.001 0.001 0.001"/>
+            <mesh filename="package://neo_mm_400/robot_model/meshes/MP-400-BODY.dae" scale="0.001 0.001 0.001"/>
         <!--cylinder length="0.381" radius="0.2545"/-->
         <!--box size="0.445 0.277 0.17"/-->
@@ -21,5 +21,5 @@
         <origin xyz="0.0 0.0 0.0" rpy="0 0 1.57" />
         <geometry>
-          <mesh filename="package://neo_simulation/robots/mm_400/meshes/MP-400-BODY.dae" scale="0.001 0.001 0.001"/>
+          <mesh filename="package://neo_mm_400/robot_model/meshes/MP-400-BODY.dae" scale="0.001 0.001 0.001"/>
           <!--cylinder length="0.381" radius="0.2545"/-->
         </geometry>

File: robot_model/urdf/xacros/mp_400_caster_wheel.xacro (robot description, xacro)
@@ -19,5 +19,5 @@
     <origin xyz="0 0 0" rpy="0 0 0" />
     <geometry>
-            <mesh filename="package://neo_simulation/robots/mp_400/meshes/MP-400-CASTER-WHEEL.dae" scale="0.001 0.001 0.001"/>
+            <mesh filename="package://neo_mm_400/robot_model/meshes/MP-400-CASTER-WHEEL.dae" scale="0.001 0.001 0.001"/>
     </geometry>
     </visual>
@@ -25,5 +25,5 @@
       <origin xyz="0 0. 0" rpy="0 0 0" />
       <geometry>
-            <mesh filename="package://neo_simulation/robots/mp_400/meshes/MP-400-CASTER-WHEEL.dae" scale="0.001 0.001 0.001"/>
+            <mesh filename="package://neo_mm_400/robot_model/meshes/MP-400-CASTER-WHEEL.dae" scale="0.001 0.001 0.001"/>
       </geometry>
     </collision>

File: robot_model/urdf/xacros/mp_400_fixed_wheel_left.xacro (robot description, xacro)
@@ -20,5 +20,5 @@
     <origin xyz="0 0 0.0" rpy="0 0 0" />
         <geometry>
-            <mesh filename="package://neo_simulation/robots/mp_400/meshes/MP-400-FIXED-WHEEL-LEFT.dae" scale="0.001 0.001 0.001"/>
+            <mesh filename="package://neo_mm_400/robot_model/meshes/MP-400-FIXED-WHEEL-LEFT.dae" scale="0.001 0.001 0.001"/>
         </geometry>
       </visual>
@@ -26,5 +26,5 @@
      <origin xyz="0. 0 0" rpy=" 0 0 0" />
       <geometry>
-            <mesh filename="package://neo_simulation/robots/mp_400/meshes/MP-400-FIXED-WHEEL-LEFT.dae" scale="0.001 0.001 0.001"/>
+            <mesh filename="package://neo_mm_400/robot_model/meshes/MP-400-FIXED-WHEEL-LEFT.dae" scale="0.001 0.001 0.001"/>
       </geometry>
     </collision>

File: robot_model/urdf/xacros/mp_400_fixed_wheel_right.xacro (robot description, xacro)
@@ -20,5 +20,5 @@
     <origin xyz="0 0 0.0" rpy="0 0 3.14" />
         <geometry>
-            <mesh filename="package://neo_simulation/robots/mp_400/meshes/MP-400-FIXED-WHEEL-RIGHT.dae" scale="0.001 0.001 0.001"/>
+            <mesh filename="package://neo_mm_400/robot_model/meshes/MP-400-FIXED-WHEEL-RIGHT.dae" scale="0.001 0.001 0.001"/>
         </geometry>
       </visual>
@@ -26,5 +26,5 @@
      <origin xyz="0. 0 0" rpy=" 0 0 0" />
       <geometry>
-            <mesh filename="package://neo_simulation/robots/mp_400/meshes/MP-400-FIXED-WHEEL-LEFT.dae" scale="0.001 0.001 0.001"/>
+            <mesh filename="package://neo_mm_400/robot_model/meshes/MP-400-FIXED-WHEEL-LEFT.dae" scale="0.001 0.001 0.001"/>
       </geometry>
     </collision>

File: robot_model/urdf/xacros/sick_laser.xacro (robot description, xacro)
@@ -18,5 +18,5 @@
 <!--       <origin xyz="0 0 -0.11" rpy="-1.57 0 3.14" />
         <geometry>
-        <mesh filename="package://neo_simulation/robots/mp_400/meshes/SICK-S300.dae" scale="0.001 0.001 0.001" />
+        <mesh filename="package://neo_mm_400/robot_model/mp_400/meshes/SICK-S300.dae" scale="0.001 0.001 0.001" />
         </geometry>
       </visual>
@@ -24,5 +24,5 @@
         <origin xyz="0 0 -0.11" rpy="-1.57 0 3.14" />
         <geometry>
-        <mesh filename="package://neo_simulation/robots/mp_400/meshes/SICK-S300.dae" scale="0.001 0.001 0.001" />
+        <mesh filename="package://neo_mm_400/robot_model/mp_400/meshes/SICK-S300.dae" scale="0.001 0.001 0.001" />
         </geometry>
       </collision> -->
@@ -30,5 +30,5 @@
  <origin xyz="-0.0 0 -0.06" rpy="1.57 0 0" />
       <geometry>
-      <mesh filename="package://neo_simulation/robots/mp_400/meshes/SICK-MICROSCAN3.dae" scale="0.001 0.001 0.001" />
+      <mesh filename="package://neo_mm_400/robot_model/meshes/SICK-MICROSCAN3.dae" scale="0.001 0.001 0.001" />
       </geometry>
       </visual>
@@ -36,5 +36,5 @@
  <origin xyz="-0.0 0 -0.06" rpy="1.57 0 0" />
       <geometry>
-        <mesh filename="package://neo_simulation/robots/mp_400/meshes/SICK-MICROSCAN3.dae" scale="0.001 0.001 0.001" />
+        <mesh filename="package://neo_mm_400/robot_model/meshes/SICK-MICROSCAN3.dae" scale="0.001 0.001 0.001" />
         </geometry>
       </collision>

Commit message: Added panda arm in the robot model

File: robot_model/mm_400.urdf.xacro (robot description, xacro)
@@ -2,19 +2,39 @@
 <!-- Materials -->
 <robot xmlns:xacro="http://www.ros.org/wiki/xacro" name="mm_400">
-<xacro:include filename="$(find neo_mm_400)/robot_model/xacros/mp_400_gazebo.xacro" />
+<xacro:include filename="$(find neo_mm_400)/robot_model/mm_400_panda/urdf/xacros/mp_400_gazebo.xacro" />
+<!-- MM400 with Panda -->
 <!--++++++++++++++++++++++++++++++base_link++++++++++++++++++++++++++++++++++++++++++++++++++++-->
 <!--++++++++++++++++++++body++++++++++++++++++++++++++++-->
-<xacro:include filename="$(find neo_mm_400)/robot_model/urdf/xacros/mp_400_body.xacro" />
+<xacro:include filename="$(find neo_mm_400)/robot_model/mm_400_panda/urdf/xacros/mp_400_body.xacro" />
 <!--+++++++++++++++++++castor_wheel_link++++++++++++++++++++++++-->
-<xacro:include filename="$(find neo_mm_400)/robot_model/urdf/xacros/mp_400_caster_wheel.xacro" />
+<xacro:include filename="$(find neo_mm_400)/robot_model/mm_400_panda/urdf/xacros/mp_400_caster_wheel.xacro" />
 <!--+++++++++++++++++++left_wheel_link++++++++++++++++++++++++-->
-<xacro:include filename="$(find neo_mm_400)/robot_model/urdf/xacros/mp_400_fixed_wheel_left.xacro" />
+<xacro:include filename="$(find neo_mm_400)/robot_model/mm_400_panda/urdf/xacros/mp_400_fixed_wheel_left.xacro" />
 <!--+++++++++++++++++++right_wheel_link++++++++++++++++++++++++-->
-<xacro:include filename="$(find neo_mm_400)/robot_model/urdf/xacros/mp_400_fixed_wheel_right.xacro" />
+<xacro:include filename="$(find neo_mm_400)/robot_model/mm_400_panda/urdf/xacros/mp_400_fixed_wheel_right.xacro" />
 <!--+++++++++++++++++++cabinet++++++++++++++++++++++++-->
-<xacro:include filename="$(find neo_mm_400)/robot_model/urdf/xacros/cabinet.xacro" />
-<xacro:include filename="$(find neo_mm_400)/robot_model/urdf/prbt_macro.xacro" />
+<xacro:include filename="$(find neo_mm_400)/robot_model/mm_400_panda/urdf/xacros/cabinet.xacro" />
  <!-- SENSORS -->
-<xacro:include filename="$(find neo_mm_400)/robot_model/urdf/xacros/sick_laser.xacro" />
+<xacro:include filename="$(find neo_mm_400)/robot_model/mm_400_panda/urdf/xacros/sick_laser.xacro" />
+<!-- Panda -->
+<xacro:include filename="$(find neo_mm_400)/robot_model/mm_400_panda/urdf/panda_arm.xacro" />
+<!-- MM400 with pilz -->
+<!-- <xacro:include filename="$(find neo_mm_400)/robot_model/mm_400_pilz/urdf/xacros/mp_400_gazebo.xacro" /> -->
+<!--++++++++++++++++++++++++++++++base_link++++++++++++++++++++++++++++++++++++++++++++++++++++-->
+<!--++++++++++++++++++++body++++++++++++++++++++++++++++-->
+<!-- <xacro:include filename="$(find neo_mm_400)/robot_model/mm_400_pilz/urdf/xacros/mp_400_body.xacro" /> -->
+<!--+++++++++++++++++++castor_wheel_link++++++++++++++++++++++++-->
+<!-- <xacro:include filename="$(find neo_mm_400)/robot_model/mm_400_pilz/urdf/xacros/mp_400_caster_wheel.xacro" /> -->
+<!--+++++++++++++++++++left_wheel_link++++++++++++++++++++++++-->
+<!-- <xacro:include filename="$(find neo_mm_400)/robot_model/mm_400_pilz/urdf/xacros/mp_400_fixed_wheel_left.xacro" /> -->
+<!--+++++++++++++++++++right_wheel_link++++++++++++++++++++++++-->
+<!-- <xacro:include filename="$(find neo_mm_400)/robot_model/mm_400_pilz/urdf/xacros/mp_400_fixed_wheel_right.xacro" /> -->
+<!--+++++++++++++++++++cabinet++++++++++++++++++++++++-->
+<!-- <xacro:include filename="$(find neo_mm_400)/robot_model/mm_400_pilz/urdf/xacros/cabinet.xacro" /> -->
+ <!-- SENSORS -->
+<!-- <xacro:include filename="$(find neo_mm_400)/robot_model/mm_400_pilz/urdf/xacros/sick_laser.xacro" /> -->
+  <!-- <xacro:include filename="$(find neo_simulation)/robots/mm_400/urdf/prbt_macro.xacro" /> -->
+<!-- Gripper -->
+<!-- <xacro:include filename="$(find schunk_description)/pg70.urdf.xacro" /> -->
   <xacro:mp_400_base name="base_link">
   </xacro:mp_400_base>
@@ -42,7 +62,15 @@
   </xacro:mm_400_cabinet>
    <!-- Robot arm -->
-  <xacro:prbt parent="cabinet_link" prefix="pilz">
+   <!-- Pilz -->
+<!--   <xacro:prbt parent="cabinet_link" prefix="pilz">
     <origin xyz="0 0 0." rpy="0 0 0" />
-  </xacro:prbt>
+  </xacro:prbt> -->
+<!-- Panda -->
+  <xacro:panda_arm parent="cabinet_link" prefix="panda">
+    <origin xyz="0 0 0." rpy="0 0 0" />
+  </xacro:panda_arm>
+<!--   <xacro:pg70 parent="pilztool0">
+    <origin xyz="0 0 0." rpy="0 0 0" />
+  </xacro:pg70> -->
   <!--+++++++++++++++++++laserscanner_link++++++++++++++++++++++++-->
   <xacro:sick_laser_v0 name="laser_1" parent="base_link" ros_topic="laser_1/scan">

Commit message: Top part has been removed

File: robot_model/mm_400.urdf.xacro (robot description, xacro)
@@ -58,7 +58,4 @@
     <origin xyz="-0. 0.26 0.074" rpy="0 0 1.57" />
   </xacro:fixed_wheel_left>
-  <xacro:mm_400_cabinet name="cabinet" parent="base_link">
-    <origin xyz="0.02 0 0.551" rpy="0 0 3.14" />
-  </xacro:mm_400_cabinet>
    <!-- Robot arm -->
    <!-- Pilz -->
@@ -67,6 +64,6 @@
   </xacro:prbt> -->
 <!-- Panda -->
-  <xacro:panda_arm parent="cabinet_link" prefix="panda">
-    <origin xyz="0 0 0." rpy="0 0 0" />
+  <xacro:panda_arm parent="base_link" prefix="panda">
+    <origin xyz="0 0 -0.0" rpy="0 0 0" />
   </xacro:panda_arm>
 <!--   <xacro:pg70 parent="pilztool0">

File: robot_model/mm_400_panda/urdf/panda_arm.xacro (robot description, xacro)
@@ -2,8 +2,8 @@
 <robot xmlns:xacro="http://www.ros.org/wiki/xacro" name="panda">
   <xacro:macro name="panda_arm" params="prefix parent *origin">
-    <joint name="cabinet_joints" type="fixed">
+    <joint name="arm_joints" type="fixed">
       <parent link="${parent}" />
       <child link = "${prefix}_link0" />
-      <origin xyz="-0.1 0.0 0.12" rpy="0.0 0.0 3.14" />
+      <origin xyz="0.125 0.0 0.381" rpy="0.0 0.0 0" />
     </joint>
   <link name="${prefix}_link0">
